File: Sat/First Project.sch (EAGLE design)
At the start: 22 parts, among them U1 ATMEGA328P_TQFP, U2 915MHz, U3 9DoF IMU, U4 3.3V/150mA

Commit message: Finished Schematic
Parts:
- removed R5, R6, R7: 10K, femtosat:RESISTOR_10KOHM0603
- removed SJ1: (no value), jumper:SJ2W
Connections:
- removed net AD0/ASO: SJ1.1
- removed net AUX_CL: U3.AUX_CL
- removed net AUX_DA: U3.AUX_DA
- removed net CS: R7.1, U3.!CS
- removed net INT: U3.INT
- removed net N$10: C3.1, U3.REGOUT
- removed net N$12: SJ1.2, U3.AD0/SDO
- removed net VDDIO: U3.VDDIO
- net 12C_SCL: no longer R5.1
- net 12C_SDA: no longer R6.1
- net 3.3V: now also U3.VDDIO; no longer R5.2, R6.2, R7.2
- net FSYNC: now also C3.1, U3.REGOUT; no longer U3.FSYNC
- net GND: now also U3.AD0/SDO, U3.AUX_CL, U3.AUX_DA, U3.FSYNC; no longer SJ1.3

Commit message: Routed Components and added a Ground Plane
Parts:
- removed J2: (no value), femtosat:CONNECTOR_2PIN
- added C4: 0.1uF, femtosat:CAPACITOR_0.1UF
- added C5: 1.0uF, femtosat:CAPACITOR_1.0UF-0603-16V-10%
- added J3: (no value), femtosat:CONNECTOR_2PIN-JST-2MM-SMT
Connections:
- removed net VBAT: J2.2, U4.IN
- new net N$2: J3.1, U4.IN
- net 3.3V: now also C4.1, C5.1
- net GND: now also C4.2, C5.2, J3.2; no longer J2.1
Changed lines of the file:
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@@
 <setting verticaltext="up"/>
 </settings>
-<grid distance="0.1" unitdist="inch" unit="inch" style="dots" multiple="1" display="yes" altdistance="0.01" altunitdist="inch" altunit="inch"/>
+<grid distance="0.1" unitdist="inch" unit="inch" style="lines" multiple="1" display="no" altdistance="0.01" altunitdist="inch" altunit="inch"/>
 <layers>
 <layer number="1" name="Top" color="4" fill="1" visible="no" active="no"/>
+<layer number="2" name="Route2" color="1" fill="3" visible="no" active="no"/>
+<layer number="3" name="Route3" color="4" fill="3" visible="no" active="no"/>
+<layer number="4" name="Route4" color="1" fill="4" visible="no" active="no"/>
+<layer number="5" name="Route5" color="4" fill="4" visible="no" active="no"/>
+<layer number="6" name="Route6" color="1" fill="8" visible="no" active="no"/>
+<layer number="7" name="Route7" color="4" fill="8" visible="no" active="no"/>
+<layer number="8" name="Route8" color="1" fill="2" visible="no" active="no"/>
+<layer number="9" name="Route9" color="4" fill="2" visible="no" active="no"/>
+<layer number="10" name="Route10" color="1" fill="7" visible="no" active="no"/>
+<layer number="11" name="Route11" color="4" fill="7" visible="no" active="no"/>
+<layer number="12" name="Route12" color="1" fill="5" visible="no" active="no"/>
+<layer number="13" name="Route13" color="4" fill="5" visible="no" active="no"/>
+<layer number="14" name="Route14" color="1" fill="6" visible="no" active="no"/>
+<layer number="15" name="Route15" color="4" fill="6" visible="no" active="no"/>
 <layer number="16" name="Bottom" color="1" fill="1" visible="no" active="no"/>
 <layer number="17" name="Pads" color="2" fill="1" visible="no" active="no"/>
@@
 <part name="P+4" library="femtosat" deviceset="3.3V" device=""/>
 <part name="B1" library="femtosat" deviceset="BATTERY_FOOTPRINT" device="" value="110mAh"/>
-<part name="J2" library="femtosat" deviceset="CONNECTOR_2PIN" device=""/>
 <part name="GND5" library="femtosat" deviceset="GND" device=""/>
 <part name="U3" library="femtosat" deviceset="MPU9250" device="" value="9DoF IMU"/>
@@
 <part name="P+9" library="femtosat" deviceset="3.3V" device=""/>
 <part name="GND10" library="femtosat" deviceset="GND" device=""/>
+<part name="C4" library="femtosat" deviceset="CAPACITOR_0.1UF" device="" value="0.1uF"/>
+<part name="C5" library="femtosat" deviceset="CAPACITOR_1.0UF" device="-0603-16V-10%" value="1.0uF"/>
+<part name="J3" library="femtosat" deviceset="CONNECTOR_2PIN" device="-JST-2MM-SMT"/>
 </parts>
 <sheets>
@@
 <instance part="P+4" gate="G$1" x="40.64" y="60.96"/>
 <instance part="B1" gate="B1" x="20.32" y="200.66"/>
-<instance part="J2" gate="G$1" x="30.48" y="198.12"/>
-<instance part="GND5" gate="1" x="43.18" y="190.5"/>
+<instance part="GND5" gate="1" x="43.18" y="203.2"/>
 <instance part="U3" gate="G$1" x="203.2" y="182.88"/>
 <instance part="C1" gate="G$1" x="160.02" y="182.88"/>
@@
 <instance part="U4" gate="U1" x="63.5" y="195.58"/>
 <instance part="P+7" gate="G$1" x="53.34" y="195.58" rot="R90"/>
-<instance part="P+8" gate="G$1" x="71.12" y="200.66" rot="R270"/>
+<instance part="P+8" gate="G$1" x="86.36" y="200.66" rot="R270"/>
 <instance part="GND9" gate="1" x="53.34" y="180.34"/>
 <instance part="P+9" gate="G$1" x="180.34" y="187.96" rot="R90"/>
 <instance part="GND10" gate="1" x="215.9" y="198.12" rot="R270"/>
+<instance part="C4" gate="G$1" x="78.74" y="195.58"/>
+<instance part="C5" gate="G$1" x="86.36" y="195.58"/>
+<instance part="J3" gate="G$1" x="30.48" y="198.12"/>
 </instances>
 <busses>
@@
 </segment>
 <segment>
-<pinref part="J2" gate="G$1" pin="1"/>
-<wire x1="38.1" y1="198.12" x2="43.18" y2="198.12" width="0.1524" layer="91"/>
-<wire x1="43.18" y1="198.12" x2="43.18" y2="193.04" width="0.1524" layer="91"/>
+<wire x1="38.1" y1="205.74" x2="43.18" y2="205.74" width="0.1524" layer="91"/>
 <pinref part="GND5" gate="1" pin="GND"/>
+<pinref part="J3" gate="G$1" pin="2"/>
+<wire x1="38.1" y1="200.66" x2="38.1" y2="205.74" width="0.1524" layer="91"/>
 </segment>
 <segment>
@@
 <pinref part="U4" gate="U1" pin="GND"/>
 <pinref part="GND9" gate="1" pin="GND"/>
-<wire x1="53.34" y1="190.5" x2="53.34" y2="182.88" width="0.1524" layer="91"/>
+<wire x1="53.34" y1="190.5" x2="53.34" y2="185.42" width="0.1524" layer="91"/>
+<pinref part="C4" gate="G$1" pin="2"/>
+<pinref part="C5" gate="G$1" pin="2"/>
+<wire x1="53.34" y1="185.42" x2="53.34" y2="182.88" width="0.1524" layer="91"/>
+<wire x1="78.74" y1="193.04" x2="81.28" y2="193.04" width="0.1524" layer="91"/>
+<wire x1="81.28" y1="193.04" x2="86.36" y2="193.04" width="0.1524" layer="91"/>
+<wire x1="81.28" y1="193.04" x2="81.28" y2="185.42" width="0.1524" layer="91"/>
+<wire x1="81.28" y1="185.42" x2="53.34" y2="185.42" width="0.1524" layer="91"/>
+<junction x="81.28" y="193.04"/>
+<junction x="53.34" y="185.42"/>
 </segment>
 <segment>
@@
 <pinref part="U4" gate="U1" pin="OUT"/>
 <pinref part="P+8" gate="G$1" pin="3.3V"/>
+<wire x1="86.36" y1="200.66" x2="78.74" y2="200.66" width="0.1524" layer="91"/>
+<pinref part="C4" gate="G$1" pin="1"/>
+<wire x1="78.74" y1="200.66" x2="71.12" y2="200.66" width="0.1524" layer="91"/>
+<junction x="78.74" y="200.66"/>
+<pinref part="C5" gate="G$1" pin="1"/>
+<junction x="86.36" y="200.66"/>
 </segment>
 <segment>
@@
 </segment>
 </net>
-<net name="VBAT" class="0">
-<segment>
-<pinref part="J2" gate="G$1" pin="2"/>
-<label x="38.1" y="200.66" size="1.778" layer="95"/>
-<pinref part="U4" gate="U1" pin="IN"/>
-<wire x1="53.34" y1="200.66" x2="38.1" y2="200.66" width="0.1524" layer="91"/>
-</segment>
-</net>
 <net name="FSYNC" class="0">
 <segment>
@@
 </segment>
 </net>
+<net name="N$2" class="0">
+<segment>
+<pinref part="U4" gate="U1" pin="IN"/>
+<wire x1="53.34" y1="200.66" x2="40.64" y2="200.66" width="0.1524" layer="91"/>
+<wire x1="40.64" y1="200.66" x2="40.64" y2="198.12" width="0.1524" layer="91"/>
+<pinref part="J3" gate="G$1" pin="1"/>
+<wire x1="40.64" y1="198.12" x2="38.1" y2="198.12" width="0.1524" layer="91"/>
+</segment>
+</net>
